File: Arduino UNO R4 Minima Extension Board.kicad_pcb (KiCad board)
At the start: 2 copper layers, 68.6 x 53.3 mm, 15 parts, among them J1 Power, J2 Analog, J3 Digital/PWM, J4 Digital/PWM, J5 Conn_01x04_Socket, J6 Conn_01x04_Socket, J7 Conn_01x05_Socket, J8 Conn_01x05_Socket, J9 Conn_01x05_Socket, U1 MCP2551-I-SN

Commit message: Add files via upload
Parts:
- removed J6: Conn_01x04_Socket, Connector_JST:JST_XA_S04B-XASK-1_1x04_P2.50mm_Horizontal
- removed J7, J8: Conn_01x05_Socket, Connector_JST:JST_XA_S05B-XASK-1_1x05_P2.50mm_Horizontal
- added J10: Conn_01x04_Socket, Connector_JST:JST_XA_S04B-XASK-1_1x04_P2.50mm_Horizontal, F.Cu at (87.5, 81.0)
- added J11: Conn_01x05_Socket, Connector_JST:JST_XA_S05B-XASK-1_1x05_P2.50mm_Horizontal, F.Cu at (55.9, 81.0)
- added J12: Conn_01x05_Socket, Connector_JST:JST_XA_S05B-XASK-1_1x05_P2.50mm_Horizontal, F.Cu at (55.9, 95.6)
- added J13: Conn_01x05_Socket, Connector_JST:JST_XA_S05B-XASK-1_1x05_P2.50mm_Horizontal, F.Cu at (55.9, 110.2)
- added J14: Conn_01x05_Socket, Connector_JST:JST_XA_S05B-XASK-1_1x05_P2.50mm_Horizontal, F.Cu at (55.9, 124.9)
- J9: value Conn_01x05_Socket -> Conn_01x04_Socket; footprint Connector_JST:JST_XA_S05B-XASK-1_1x05_P2.50mm_Horizontal -> Connector_JST:JST_XA_S04B-XASK-1_1x04_P2.50mm_Horizontal
- moved J9 33.2 mm to (73.0, 81.0)
- moved J5 30.5 mm to (76.8, 108.0)
- moved U1 4.00 mm to (73.7, 94.5)
- moved R1 4.00 mm to (79.9, 92.4)
- renumbered J3 to J2, J2 to J3
Connections:
- J5 pad 2: /CANH -> /SCL/A5
- J5 pad 3: /CANL -> /SDA/A4
- J9 pad 1: /9 -> +5V
- J9 pad 2: /10 -> /CANH
- J9 pad 3: /11 -> /CANL
- J9 pad 4: /12 -> GND
- U1 pad 1: /*3 -> /CAN_TX
- U1 pad 4: /4 -> /CAN_RX
